File: hardware/receiver/receiver.sch (KiCad schematic (older format))
At the start: 19 parts, among them J1 Input, J3 LED_OUT

Commit message: Add RXCLK to D9 connection for Leonardo PCINT5.
Connections:
- wire segments 71 -> 73
- no-connect marks 17 -> 16
Changed lines of the file:
@@
 Sheet 1 1
 Title "DMX Demonstrator - Receiver (DMX-RX1)"
-Date "2020-12-28"
+Date "2020-12-30"
 Rev "1.2"
 Comp "Crazy Giraffe Software"
@@
 NoConn ~ 6200 2850
 NoConn ~ 6200 2950
-Text Label 6250 3350 0    50   ~ 0
+Text Label 6200 3350 0    50   ~ 0
 ~DIM3
-Text Label 6250 3450 0    50   ~ 0
+Text Label 6200 3450 0    50   ~ 0
 ~DIM2
-Text Label 6250 3850 0    50   ~ 0
+Text Label 6200 3850 0    50   ~ 0
 ~DIM1
-Text Label 6250 3950 0    50   ~ 0
+Text Label 6200 3950 0    50   ~ 0
 ~DIM0
 NoConn ~ 5200 3250
 Wire Wire Line
-	6200 4150 6450 4150
-Wire Wire Line
-	6450 4150 6450 4950
-Wire Wire Line
-	6200 4050 6550 4050
-Wire Wire Line
-	6550 4050 6550 5150
-Wire Wire Line
-	6650 5150 7050 5150
-Wire Wire Line
-	6750 4800 7050 4800
-Wire Wire Line
-	6850 4450 7050 4450
+	6200 4150 6550 4150
+Wire Wire Line
+	6550 4150 6550 4950
+Wire Wire Line
+	6200 4050 6650 4050
+Wire Wire Line
+	6650 4050 6650 5150
+Wire Wire Line
+	6750 5150 7150 5150
+Wire Wire Line
+	6850 4800 7150 4800
+Wire Wire Line
+	6950 4450 7150 4450
 $Comp
 L Device:LED D3
 U 1 1 5F3BEC78
-P 7200 4100
-F 0 "D3" H 7191 4316 50  0000 C CNN
-F 1 "DIM3" H 7191 4225 50  0000 C CNN
-F 2 "LED_THT:LED_D5.0mm" H 7200 4100 50  0001 C CNN
-F 3 "~" H 7200 4100 50  0001 C CNN
-	1    7200 4100
+P 7300 4100
+F 0 "D3" H 7291 4316 50  0000 C CNN
+F 1 "DIM3" H 7291 4225 50  0000 C CNN
+F 2 "LED_THT:LED_D5.0mm" H 7300 4100 50  0001 C CNN
+F 3 "~" H 7300 4100 50  0001 C CNN
+	1    7300 4100
 	-1   0    0    -1
 $EndComp
@@
 L Device:R_US R3
 U 1 1 5F3BECD4
-P 7600 4100
-F 0 "R3" V 7395 4100 50  0000 C CNN
-F 1 "330" V 7486 4100 50  0000 C CNN
-F 2 "Resistor_THT:R_Axial_DIN0207_L6.3mm_D2.5mm_P10.16mm_Horizontal" V 7640 4090 50  0001 C CNN
-F 3 "~" H 7600 4100 50  0001 C CNN
-	1    7600 4100
+P 7700 4100
+F 0 "R3" V 7495 4100 50  0000 C CNN
+F 1 "330" V 7586 4100 50  0000 C CNN
+F 2 "Resistor_THT:R_Axial_DIN0207_L6.3mm_D2.5mm_P10.16mm_Horizontal" V 7740 4090 50  0001 C CNN
+F 3 "~" H 7700 4100 50  0001 C CNN
+	1    7700 4100
 	0    1    1    0
 $EndComp
@@
 L Device:LED D4
 U 1 1 5F3BFD29
-P 7200 4450
-F 0 "D4" H 7191 4666 50  0000 C CNN
-F 1 "DIM2" H 7191 4575 50  0000 C CNN
-F 2 "LED_THT:LED_D5.0mm" H 7200 4450 50  0001 C CNN
-F 3 "~" H 7200 4450 50  0001 C CNN
-	1    7200 4450
+P 7300 4450
+F 0 "D4" H 7291 4666 50  0000 C CNN
+F 1 "DIM2" H 7291 4575 50  0000 C CNN
+F 2 "LED_THT:LED_D5.0mm" H 7300 4450 50  0001 C CNN
+F 3 "~" H 7300 4450 50  0001 C CNN
+	1    7300 4450
 	-1   0    0    -1
 $EndComp
@@
 L Device:R_US R4
 U 1 1 5F3BFD2F
-P 7600 4450
-F 0 "R4" V 7395 4450 50  0000 C CNN
-F 1 "330" V 7486 4450 50  0000 C CNN
-F 2 "Resistor_THT:R_Axial_DIN0207_L6.3mm_D2.5mm_P10.16mm_Horizontal" V 7640 4440 50  0001 C CNN
-F 3 "~" H 7600 4450 50  0001 C CNN
-	1    7600 4450
+P 7700 4450
+F 0 "R4" V 7495 4450 50  0000 C CNN
+F 1 "330" V 7586 4450 50  0000 C CNN
+F 2 "Resistor_THT:R_Axial_DIN0207_L6.3mm_D2.5mm_P10.16mm_Horizontal" V 7740 4440 50  0001 C CNN
+F 3 "~" H 7700 4450 50  0001 C CNN
+	1    7700 4450
 	0    1    1    0
 $EndComp
@@
 L Device:LED D5
 U 1 1 5F3C1D16
-P 7200 4800
-F 0 "D5" H 7191 5016 50  0000 C CNN
-F 1 "DIM1" H 7191 4925 50  0000 C CNN
-F 2 "LED_THT:LED_D5.0mm" H 7200 4800 50  0001 C CNN
-F 3 "~" H 7200 4800 50  0001 C CNN
-	1    7200 4800
+P 7300 4800
+F 0 "D5" H 7291 5016 50  0000 C CNN
+F 1 "DIM1" H 7291 4925 50  0000 C CNN
+F 2 "LED_THT:LED_D5.0mm" H 7300 4800 50  0001 C CNN
+F 3 "~" H 7300 4800 50  0001 C CNN
+	1    7300 4800
 	-1   0    0    -1
 $EndComp
@@
 L Device:R_US R5
 U 1 1 5F3C1D1C
-P 7600 4800
-F 0 "R5" V 7395 4800 50  0000 C CNN
-F 1 "330" V 7486 4800 50  0000 C CNN
-F 2 "Resistor_THT:R_Axial_DIN0207_L6.3mm_D2.5mm_P10.16mm_Horizontal" V 7640 4790 50  0001 C CNN
-F 3 "~" H 7600 4800 50  0001 C CNN
-	1    7600 4800
+P 7700 4800
+F 0 "R5" V 7495 4800 50  0000 C CNN
+F 1 "330" V 7586 4800 50  0000 C CNN
+F 2 "Resistor_THT:R_Axial_DIN0207_L6.3mm_D2.5mm_P10.16mm_Horizontal" V 7740 4790 50  0001 C CNN
+F 3 "~" H 7700 4800 50  0001 C CNN
+	1    7700 4800
 	0    1    1    0
 $EndComp
@@
 L Device:LED D6
 U 1 1 5F3C1D22
-P 7200 5150
-F 0 "D6" H 7191 5366 50  0000 C CNN
-F 1 "DIM0" H 7191 5275 50  0000 C CNN
-F 2 "LED_THT:LED_D5.0mm" H 7200 5150 50  0001 C CNN
-F 3 "~" H 7200 5150 50  0001 C CNN
-	1    7200 5150
+P 7300 5150
+F 0 "D6" H 7291 5366 50  0000 C CNN
+F 1 "DIM0" H 7291 5275 50  0000 C CNN
+F 2 "LED_THT:LED_D5.0mm" H 7300 5150 50  0001 C CNN
+F 3 "~" H 7300 5150 50  0001 C CNN
+	1    7300 5150
 	-1   0    0    -1
 $EndComp
@@
 L Device:R_US R6
 U 1 1 5F3C1D28
-P 7600 5150
-F 0 "R6" V 7395 5150 50  0000 C CNN
-F 1 "330" V 7486 5150 50  0000 C CNN
-F 2 "Resistor_THT:R_Axial_DIN0207_L6.3mm_D2.5mm_P10.16mm_Horizontal" V 7640 5140 50  0001 C CNN
-F 3 "~" H 7600 5150 50  0001 C CNN
-	1    7600 5150
+P 7700 5150
+F 0 "R6" V 7495 5150 50  0000 C CNN
+F 1 "330" V 7586 5150 50  0000 C CNN
+F 2 "Resistor_THT:R_Axial_DIN0207_L6.3mm_D2.5mm_P10.16mm_Horizontal" V 7740 5140 50  0001 C CNN
+F 3 "~" H 7700 5150 50  0001 C CNN
+	1    7700 5150
 	0    1    1    0
 $EndComp
 Wire Wire Line
-	7750 4800 7950 4800
-Wire Wire Line
-	7350 5150 7450 5150
-Wire Wire Line
-	7750 5150 7950 5150
-Wire Wire Line
-	7350 4100 7450 4100
-Wire Wire Line
-	7750 4100 7950 4100
-Wire Wire Line
-	7350 4450 7450 4450
-Wire Wire Line
-	7750 4450 7950 4450
-Wire Wire Line
-	7350 4800 7450 4800
-Connection ~ 7950 4800
-Wire Wire Line
-	7950 4800 7950 5150
-Connection ~ 7950 4450
-Wire Wire Line
-	7950 4450 7950 4800
-Wire Wire Line
-	7950 4100 7950 4450
+	7850 4800 8050 4800
+Wire Wire Line
+	7450 5150 7550 5150
+Wire Wire Line
+	7850 5150 8050 5150
+Wire Wire Line
+	7450 4100 7550 4100
+Wire Wire Line
+	7850 4100 8050 4100
+Wire Wire Line
+	7450 4450 7550 4450
+Wire Wire Line
+	7850 4450 8050 4450
+Wire Wire Line
+	7450 4800 7550 4800
+Connection ~ 8050 4800
+Wire Wire Line
+	8050 4800 8050 5150
+Connection ~ 8050 4450
+Wire Wire Line
+	8050 4450 8050 4800
+Wire Wire Line
+	8050 4100 8050 4450
 $Comp
 L Connector:Screw_Terminal_01x05 J3
 U 1 1 5F42826E
-P 8250 3550
-F 0 "J3" H 8330 3592 50  0000 L CNN
-F 1 "LED_OUT" H 8330 3501 50  0000 L CNN
-F 2 "Connector_Phoenix_MSTB:PhoenixContact_MSTBA_2,5_5-G-5,08_1x05_P5.08mm_Horizontal" H 8250 3550 50  0001 C CNN
-F 3 "~" H 8250 3550 50  0001 C CNN
-	1    8250 3550
+P 8350 3550
+F 0 "J3" H 8430 3592 50  0000 L CNN
+F 1 "LED_OUT" H 8430 3501 50  0000 L CNN
+F 2 "Connector_Phoenix_MSTB:PhoenixContact_MSTBA_2,5_5-G-5,08_1x05_P5.08mm_Horizontal" H 8350 3550 50  0001 C CNN
+F 3 "~" H 8350 3550 50  0001 C CNN
+	1    8350 3550
 	1    0    0    1
 $EndComp
@@
 L power:GND #PWR0113
 U 1 1 5F443F49
-P 7950 5250
-F 0 "#PWR0113" H 7950 5000 50  0001 C CNN
-F 1 "GND" H 7955 5077 50  0000 C CNN
-F 2 "" H 7950 5250 50  0001 C CNN
-F 3 "" H 7950 5250 50  0001 C CNN
-	1    7950 5250
+P 8050 5250
+F 0 "#PWR0113" H 8050 5000 50  0001 C CNN
+F 1 "GND" H 8055 5077 50  0000 C CNN
+F 2 "" H 8050 5250 50  0001 C CNN
+F 3 "" H 8050 5250 50  0001 C CNN
+	1    8050 5250
 	1    0    0    -1
 $EndComp
 Wire Wire Line
-	8050 3750 7950 3750
-Text Label 6250 4050 0    50   ~ 0
+	8150 3750 8050 3750
+Text Label 6200 4050 0    50   ~ 0
 RX
-Text Label 6250 4150 0    50   ~ 0
+Text Label 6200 4150 0    50   ~ 0
 RXCLK
 NoConn ~ 5800 2450
@@
 D0-D4\nReserved\nFor DMX\nShield
 Wire Wire Line
-	6950 4100 7050 4100
+	7050 4100 7150 4100
 $Comp
 L power:+5V #PWR0104
@@
 	6550 7350 6550 7450
 Wire Wire Line
-	7950 5250 7950 5150
-Connection ~ 7950 5150
-Wire Wire Line
-	7950 3750 7950 4100
-Connection ~ 7950 4100
-Wire Wire Line
-	4150 5150 6550 5150
-Wire Wire Line
-	4150 4950 6450 4950
-Connection ~ 6650 3950
-Wire Wire Line
-	6650 3950 6650 5150
-Connection ~ 6750 3850
-Wire Wire Line
-	6750 3850 6750 4800
-Wire Wire Line
-	6750 3550 8050 3550
-Wire Wire Line
-	6650 3650 6650 3950
-Wire Wire Line
-	6750 3550 6750 3850
-Wire Wire Line
-	6850 4450 6850 3450
-Connection ~ 6850 3450
-Wire Wire Line
-	6850 3450 8050 3450
-Wire Wire Line
-	6650 3650 8050 3650
-Wire Wire Line
-	6200 3350 6950 3350
-Wire Wire Line
-	6200 3450 6850 3450
-Wire Wire Line
-	6200 3950 6650 3950
-Wire Wire Line
-	6200 3850 6750 3850
+	8050 5250 8050 5150
+Connection ~ 8050 5150
+Wire Wire Line
+	8050 3750 8050 4100
+Connection ~ 8050 4100
+Wire Wire Line
+	4150 5150 6650 5150
+Wire Wire Line
+	4150 4950 6550 4950
+Connection ~ 6750 3950
+Wire Wire Line
+	6750 3950 6750 5150
+Connection ~ 6850 3850
+Wire Wire Line
+	6850 3850 6850 4800
+Wire Wire Line
+	6850 3550 8150 3550
+Wire Wire Line
+	6750 3650 6750 3950
+Wire Wire Line
+	6850 3550 6850 3850
+Wire Wire Line
+	6950 4450 6950 3450
+Connection ~ 6950 3450
+Wire Wire Line
+	6950 3450 8150 3450
+Wire Wire Line
+	6750 3650 8150 3650
 NoConn ~ 6200 3650
-NoConn ~ 6200 3750
-Wire Wire Line
-	6950 4100 6950 3350
-Wire Wire Line
-	6950 3350 8050 3350
-Connection ~ 6950 3350
+Wire Wire Line
+	7050 4100 7050 3350
+Wire Wire Line
+	7050 3350 8150 3350
 $Comp
 L Device:LED D7
@@
 Wire Wire Line
 	4600 3750 5200 3750
+Connection ~ 7050 3350
+Wire Wire Line
+	6550 4150 6550 3750
+Wire Wire Line
+	6550 3750 6200 3750
+Connection ~ 6550 4150
+Wire Wire Line
+	6200 3950 6750 3950
+Wire Wire Line
+	6200 3850 6850 3850
+Wire Wire Line
+	6200 3450 6950 3450
+Wire Wire Line
+	6200 3350 7050 3350
 $EndSCHEMATC
