File: hardware/control-pro/transmitter/transmitter.sch (KiCad schematic (older format))
At the start: 8 parts, among them J1 Output, J2 INPUT

Commit message: DMX-TX2 V1.1: - Fixed shield footprint - Moved Clock LED to avoid Arduino ICSP connector. - Relabeled the clock fast and slow LED connections in the   schematic to match the board layout. - Added Fcu power plane - Redid Fcu layout - Added rounded corners
Parts:
- A1: footprint Module:Arduino_UNO_R3 -> footprints:ARDUINO_R3_NO_HOLES
Changed lines of the file:
@@
 Sheet 1 1
 Title "DMX Demonstrator - Transmitter for Control-Pro (DMX-TX2)"
-Date "2020-09-25"
-Rev "1.0"
+Date "2020-12-30"
+Rev "1.1"
 Comp "Crazy Giraffe Software"
 Comment1 ""
@@
 F 0 "A1" H 6000 4400 50  0000 C CNN
 F 1 "Arduino_UNO_R3" H 5750 4300 50  0000 C CNN
-F 2 "Module:Arduino_UNO_R3" H 6350 2300 50  0001 L CNN
+F 2 "footprints:ARDUINO_R3_NO_HOLES" H 6350 2300 50  0001 L CNN
 F 3 "https://www.arduino.cc/en/Main/arduinoBoardUno" H 6000 4400 50  0001 C CNN
 	1    6200 3350
@@
 	6700 3650 7050 3650
 Text Label 6750 3650 0    50   ~ 0
+~CLK_SLO
+Text Label 6750 3550 0    50   ~ 0
 ~CLK_FST
-Text Label 6750 3550 0    50   ~ 0
-~CLK_SLO
 $Comp
 L Device:R_US R?

Commit message: TX2: - Added buffer to drive LEDs - Added decoupling capacitors - Fixed dimmer traces on PCB
DMX-CPC*:
- Switched to horizontal 16 pin connectors since vertical was too tall with a cable plugged in
- Swapped the clock speed and step switches to match the order on the TX1
- Swapped the data and clock LEDs to match the order on the TX1

DMX-CPD*:
- Split dimmer controls out to its own PCB
- Added 2nd 16 pin connector to daisy chain with DMX-CPC*.
- Switched to horizontal 16 pin connectors since vertical was too tall with a cable plugged in

Updated readmes with parts, board links.
Parts:
- added C1: 0.1uF, Capacitor_THT:C_Disc_D3.0mm_W1.6mm_P2.50mm, symbol Device:C_Small
- added C2: 10uF, Capacitor_THT:CP_Radial_D4.0mm_P1.50mm, symbol Device:CP1
- added U1: 74LS365, Package_DIP:DIP-16_W7.62mm, symbol 74xx:74LS365
Connections:
- net labels added: CLOCK, DATA, HWD_DT
- wire segments 60 -> 77
- no-connect marks 13 -> 15
