File: hardware/display-pro/display-pro.sch (KiCad schematic (older format))
At the start: 16 parts, among them J2 POWER, J3 Input, J4 Output, J5 Clock, J6 Data, Q1 FQP30N06L, Q2 FQP30N06L

Commit message: Prototype version of DMX, Analog, and PWM IO Modules and both TX and RX IO interfaces.
Make io-analog a stackable family
io-analog-core handles D to A
io-analog-voltage handles voltage output
io-analog-pwm handles pwm output for leds, drive display pro

Refactor display-pro to work with io-analog-pwm
Add correct coax power connector

Move TX2 to tx-io
Parts:
- removed R3, R4: R?, Resistor_THT:R_Axial_DIN0411_L9.9mm_D3.6mm_P15.24mm_Horizontal, symbol Device:R_US
- added J4: Power, Connectors:POWER_JACK_PTH_BREAD, symbol CrazyGiraffe_DMXDemonstrator:POWER_JACKPTH_BREAD
- J3: renamed from J2; value POWER -> Power
- J5: value Clock -> C Out
- J6: value Data -> D Out
- Q1, Q2: symbol SparkFun-DiscreteSemi:MOSFET-NCH-FQP30N06L -> CrazyGiraffe_DMXDemonstrator:MOSFET-NCH-FQP30N06L
- renumbered J3 to J1, J4 to J2
Connections:
- net labels added: C, D
- net labels removed: CLOCK, DATA
- wire segments 53 -> 40
Other:
- note removed: "Cut trace to\nuse resistor"
- moved on the sheet: D1
