File: hardware/control-pro/clock-control/clock-control.sch (KiCad schematic (older format))
At the start: 17 parts, among them J1 OUTPUT, J2 INPUT, SW1 CLOCK_SPEED, SW2 CLOCK_STEP

Commit message: TX2: - Added buffer to drive LEDs - Added decoupling capacitors - Fixed dimmer traces on PCB
DMX-CPC*:
- Switched to horizontal 16 pin connectors since vertical was too tall with a cable plugged in
- Swapped the clock speed and step switches to match the order on the TX1
- Swapped the data and clock LEDs to match the order on the TX1

DMX-CPD*:
- Split dimmer controls out to its own PCB
- Added 2nd 16 pin connector to daisy chain with DMX-CPC*.
- Switched to horizontal 16 pin connectors since vertical was too tall with a cable plugged in

Updated readmes with parts, board links.
Parts:
- J1, J2: footprint Connector_IDC:IDC-Header_2x08_P2.54mm_Vertical -> Connector_IDC:IDC-Header_2x08_P2.54mm_Horizontal
Changed lines of the file:
@@
 Sheet 1 1
 Title "DMX Demonstrator - Control-Pro Clock (DMX-CPCB)"
-Date "2022-09-06"
+Date "2023-02-11"
 Rev "1.2"
 Comp "Crazy Giraffe Software"
@@
 F 0 "J1" H 6000 3917 50  0000 C CNN
 F 1 "OUTPUT" H 6000 3826 50  0000 C CNN
-F 2 "Connector_IDC:IDC-Header_2x08_P2.54mm_Vertical" H 5950 3400 50  0001 C CNN
+F 2 "Connector_IDC:IDC-Header_2x08_P2.54mm_Horizontal" H 5950 3400 50  0001 C CNN
 F 3 "~" H 5950 3400 50  0001 C CNN
 	1    5950 3400
@@
 F 0 "J2" H 4200 3917 50  0000 C CNN
 F 1 "INPUT" H 4200 3826 50  0000 C CNN
-F 2 "Connector_IDC:IDC-Header_2x08_P2.54mm_Vertical" H 4150 3400 50  0001 C CNN
+F 2 "Connector_IDC:IDC-Header_2x08_P2.54mm_Horizontal" H 4150 3400 50  0001 C CNN
 F 3 "~" H 4150 3400 50  0001 C CNN
 	1    4150 3400
