File: hardware/control-pro/dimmer-control/dimmer-control.kicad_pcb (KiCad board)
At the start: 2 copper layers, 100 x 90 mm, 22 parts, among them J1 OUTPUT, J2 INPUT

Commit message: Add copper pours to faceplates.
Other:
- board text added: "DMX-CPDB, Rev 1.3 Crazy Giraffe Software"
- board text removed: "DMX-CPDB, Rev 1.2 Crazy Giraffe Software"
Changed lines of the file:
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@@
   (title_block
     (title "DMX Demonstrator - Control-Pro Dimmer (DMX-CPDB)")
-    (date 2023-02-11)
-    (rev 1.2)
+    (date 2023-12-04)
+    (rev 1.3)
     (company "Crazy Giraffe Software")
     (comment 2 "Designed by: SparkyBobo")
@@
     (effects (font (size 1.5 1.5) (thickness 0.3)))
   )
-  (gr_text "DMX-CPDB, Rev 1.2\nCrazy Giraffe Software" (at 160.414 136.102) (layer B.SilkS)
+  (gr_text "DMX-CPDB, Rev 1.3\nCrazy Giraffe Software" (at 160.414 136.102) (layer B.SilkS)
     (effects (font (size 1 1) (thickness 0.15)) (justify mirror))
   )
