File: hardware/control-pro/dimmer-control/dimmer-control.sch (KiCad schematic (older format))
At the start: 20 parts, among them J1 OUTPUT, J2 INPUT

Commit message: TX2: - Added buffer to drive LEDs - Added decoupling capacitors - Fixed dimmer traces on PCB
DMX-CPC*:
- Switched to horizontal 16 pin connectors since vertical was too tall with a cable plugged in
- Swapped the clock speed and step switches to match the order on the TX1
- Swapped the data and clock LEDs to match the order on the TX1

DMX-CPD*:
- Split dimmer controls out to its own PCB
- Added 2nd 16 pin connector to daisy chain with DMX-CPC*.
- Switched to horizontal 16 pin connectors since vertical was too tall with a cable plugged in

Updated readmes with parts, board links.
Parts:
- D8: value LED -> ACTIVE
- J1, J2: footprint Connector_IDC:IDC-Header_2x08_P2.54mm_Vertical -> Connector_IDC:IDC-Header_2x08_P2.54mm_Horizontal
Changed lines of the file:
@@
 Sheet 1 1
 Title "DMX Demonstrator - Control-Pro Dimmer (DMX-CPDB)"
-Date "2022-09-06"
+Date "2023-02-11"
 Rev "1.2"
 Comp "Crazy Giraffe Software"
@@
 F 0 "J1" H 4700 4117 50  0000 C CNN
 F 1 "OUTPUT" H 4700 4026 50  0000 C CNN
-F 2 "Connector_IDC:IDC-Header_2x08_P2.54mm_Vertical" H 4650 3600 50  0001 C CNN
+F 2 "Connector_IDC:IDC-Header_2x08_P2.54mm_Horizontal" H 4650 3600 50  0001 C CNN
 F 3 "~" H 4650 3600 50  0001 C CNN
 	1    4650 3600
@@
 F 0 "J2" H 7100 4117 50  0000 C CNN
 F 1 "INPUT" H 7100 4026 50  0000 C CNN
-F 2 "Connector_IDC:IDC-Header_2x08_P2.54mm_Vertical" H 7050 3600 50  0001 C CNN
+F 2 "Connector_IDC:IDC-Header_2x08_P2.54mm_Horizontal" H 7050 3600 50  0001 C CNN
 F 3 "~" H 7050 3600 50  0001 C CNN
 	1    7050 3600
@@
 P 4650 2600
 F 0 "D8" H 4641 2816 50  0000 C CNN
-F 1 "LED" H 4641 2725 50  0000 C CNN
+F 1 "ACTIVE" H 4641 2725 50  0000 C CNN
 F 2 "LED_THT:LED_D5.0mm" H 4650 2600 50  0001 C CNN
 F 3 "~" H 4650 2600 50  0001 C CNN
